File: jetson-nano-ppoe/jetson-nano-ppoe.sch (KiCad schematic (older format))
At the start: 31 parts, among them IC1 TPS566238PRQFR, J1 Conn_01x02, J2 Conn_02x05_Odd_Even, J3 Conn_02x02_Odd_Even, Q1 Q_PMOS_GSD, Q2 Q_PMOS_GSD, Q4 Q_NMOS_DUAL

Commit message: jetson-nano-ppoe more floorplan and spice model attempt
Parts:
- added V_CONN1, V_TR2: VDC, symbol Simulation_SPICE:VDC
- D1, D2: Spice_Lib_File (none) -> /Users/ihartwig/repos/KiCad-Spice-Library/Models/Diode/led.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; Spice_Model (none) -> LED_GENERAL; Spice_Netlist_Enabled (none) -> Y; Spice_Primitive (none) -> D
- D3, D4: Mfg (none) -> Nexperia; Mfg PN (none) -> BZX384-C5V1,115; Spice_Lib_File (none) -> /Users/ihartwig/repos/KiCad-Spice-Library/Models/Diode/zene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; Spice_Model (none) -> DI_1N4733A; Spice_Netlist_Enabled (none) -> Y; Spice_Primitive (none) -> X
- Q1, Q2: Spice_Lib_File (none) -> /Users/ihartwig/repos/KiCad-Spice-Library/Models/Transistor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; Spice_Model (none) -> cmosp; Spice_Netlist_Enabled (none) -> Y; Spice_Primitive (none) -> M
- Q4: Spice_Lib_File (none) -> /Users/ihartwig/repos/KiCad-Spice-Library/Models/Transistor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; Spice_Model (none) -> cmosn; Spice_Netlist_Enabled (none) -> Y; Spice_Primitive (none) -> M
- RN1, RN2: symbol Device:R_Pack04_SIP_Split -> frc-on-ftc-hw-special:R_Pack04_SMD_Split
Connections:
- wire segments 152 -> 164
Changed lines of the file:
@@
 F 2 "" H 4500 3250 50  0001 C CNN
 F 3 "" H 4500 3250 50  0001 C CNN
+F 4 "I" H 4500 3250 50  0001 C CNN "Spice_Primitive"
+F 5 "N" H 4500 3250 50  0001 C CNN "Spice_Netlist_Enabled"
 	1    4500 3250
 	1    0    0    -1
@@
 F 6 "Diodes Incorporated" V 3300 3450 50  0001 C CNN "Mfg 2"
 F 7 "DMG2305UX-7" V 3300 3450 50  0001 C CNN "Mfg PN 2"
+F 8 "M" H 3300 3450 50  0001 C CNN "Spice_Primitive"
+F 9 "cmosp" H 3300 3450 50  0001 C CNN "Spice_Model"
+F 10 "Y" H 3300 3450 50  0001 C CNN "Spice_Netlist_Enabled"
+F 11 "/Users/ihartwig/repos/KiCad-Spice-Library/Models/Transistor/FET/cmos.lib" H 3300 3450 50  0001 C CNN "Spice_Lib_File"
 	1    3300 3450
 	0    -1   -1   0
@@
 F 2 "LED_SMD:LED_0603_1608Metric" V 4150 3600 50  0001 C CNN
 F 3 "~" V 4150 3600 50  0001 C CNN
+F 4 "D" H 4150 3600 50  0001 C CNN "Spice_Primitive"
+F 5 "LED_GENERAL" H 4150 3600 50  0001 C CNN "Spice_Model"
+F 6 "Y" H 4150 3600 50  0001 C CNN "Spice_Netlist_Enabled"
+F 7 "/Users/ihartwig/repos/KiCad-Spice-Library/Models/Diode/led.lib" H 4150 3600 50  0001 C CNN "Spice_Lib_File"
 	1    4150 3600
 	0    -1   -1   0
 $EndComp
 $Comp
-L Device:R_Pack04_SIP_Split RN1
+L frc-on-ftc-hw-special:R_Pack04_SMD_Split RN1
 U 4 1 626CB9B3
 P 3700 4100
@@
 $EndComp
 $Comp
-L Device:R_Pack04_SIP_Split RN1
+L frc-on-ftc-hw-special:R_Pack04_SMD_Split RN1
 U 3 1 626CC091
 P 4150 4100
@@
 $EndComp
 $Comp
-L Device:R_Pack04_SIP_Split RN2
+L frc-on-ftc-hw-special:R_Pack04_SMD_Split RN2
 U 3 1 626CC5BF
 P 4150 6450
@@
 	1    0    0    -1
 $EndComp
-$Comp
-L Device:R_Pack04_SIP_Split RN1
-U 1 1 626CC9C4
-P 2700 3600
-F 0 "RN1" H 2788 3646 50  0000 L CNN
-F 1 "10k" H 2788 3555 50  0000 L CNN
-F 2 "Resistor_SMD:R_Array_Convex_4x1206" V 2620 3600 50  0001 C CNN
-F 3 "http://www.vishay.com/docs/31509/csc.pdf" H 2700 3600 50  0001 C CNN
-F 4 "Yaego" H 2700 3600 50  0001 C CNN "Mfg"
-F 5 "YC164-JR-0710KL" H 2700 3600 50  0001 C CNN "Mfg PN"
-	1    2700 3600
-	1    0    0    -1
-$EndComp
 Wire Wire Line
 	3700 3950 3700 3850
@@
 F 2 "" H 3700 4950 50  0001 C CNN
 F 3 "" H 3700 4950 50  0001 C CNN
+F 4 "I" H 3700 4950 50  0001 C CNN "Spice_Primitive"
+F 5 "N" H 3700 4950 50  0001 C CNN "Spice_Netlist_Enabled"
 	1    3700 4950
 	1    0    0    -1
@@
 F 2 "Diode_SMD:D_SOD-323_HandSoldering" H 3700 3600 50  0001 C CNN
 F 3 "~" H 3700 3600 50  0001 C CNN
+F 4 "X" H 3700 3600 50  0001 C CNN "Spice_Primitive"
+F 5 "DI_1N4733A" H 3700 3600 50  0001 C CNN "Spice_Model"
+F 6 "Y" H 3700 3600 50  0001 C CNN "Spice_Netlist_Enabled"
+F 7 "/Users/ihartwig/repos/KiCad-Spice-Library/Models/Diode/zener.lib" H 3700 3600 50  0001 C CNN "Spice_Lib_File"
+F 8 "Nexperia" V 3700 3600 50  0001 C CNN "Mfg"
+F 9 "BZX384-C5V1,115" V 3700 3600 50  0001 C CNN "Mfg PN"
 	1    3700 3600
 	0    1    1    0
@@
 F 2 "" H 4550 5600 50  0001 C CNN
 F 3 "" H 4550 5600 50  0001 C CNN
+F 4 "I" H 4550 5600 50  0001 C CNN "Spice_Primitive"
+F 5 "N" H 4550 5600 50  0001 C CNN "Spice_Netlist_Enabled"
 	1    4550 5600
 	1    0    0    -1
@@
 F 6 "Diodes Incorporated" V 3300 5800 50  0001 C CNN "Mfg 2"
 F 7 "DMG2305UX-7" V 3300 5800 50  0001 C CNN "Mfg PN 2"
+F 8 "M" H 3300 5800 50  0001 C CNN "Spice_Primitive"
+F 9 "cmosp" H 3300 5800 50  0001 C CNN "Spice_Model"
+F 10 "Y" H 3300 5800 50  0001 C CNN "Spice_Netlist_Enabled"
+F 11 "/Users/ihartwig/repos/KiCad-Spice-Library/Models/Transistor/FET/cmos.lib" H 3300 5800 50  0001 C CNN "Spice_Lib_File"
 	1    3300 5800
 	0    -1   -1   0
@@
 F 2 "LED_SMD:LED_0603_1608Metric" V 4150 5950 50  0001 C CNN
 F 3 "~" V 4150 5950 50  0001 C CNN
+F 4 "D" H 4150 5950 50  0001 C CNN "Spice_Primitive"
+F 5 "LED_GENERAL" H 4150 5950 50  0001 C CNN "Spice_Model"
+F 6 "Y" H 4150 5950 50  0001 C CNN "Spice_Netlist_Enabled"
+F 7 "/Users/ihartwig/repos/KiCad-Spice-Library/Models/Diode/led.lib" H 4150 5950 50  0001 C CNN "Spice_Lib_File"
 	1    4150 5950
 	0    -1   -1   0
 $EndComp
 $Comp
-L Device:R_Pack04_SIP_Split RN2
+L frc-on-ftc-hw-special:R_Pack04_SMD_Split RN2
 U 2 1 627B81AE
 P 2700 6450
@@
 $EndComp
 $Comp
-L Device:R_Pack04_SIP_Split RN2
+L frc-on-ftc-hw-special:R_Pack04_SMD_Split RN2
 U 1 1 627B81B4
 P 2700 5950
@@
 F 5 "YC164-JR-0710KL" H 2700 5950 50  0001 C CNN "Mfg PN"
 	1    2700 5950
-	1    0    0    -1
-$EndComp
-$Comp
-L Device:R_Pack04_SIP_Split RN2
+	1    0    0    1
+$EndComp
+$Comp
+L frc-on-ftc-hw-special:R_Pack04_SMD_Split RN2
 U 4 1 627B81BA
 P 3700 6450
@@
 $EndComp
 $Comp
-L Device:R_Pack04_SIP_Split RN1
+L frc-on-ftc-hw-special:R_Pack04_SMD_Split RN1
 U 2 1 627B81C0
 P 2700 4100
@@
 F 2 "" H 3700 7300 50  0001 C CNN
 F 3 "" H 3700 7300 50  0001 C CNN
+F 4 "I" H 3700 7300 50  0001 C CNN "Spice_Primitive"
+F 5 "N" H 3700 7300 50  0001 C CNN "Spice_Netlist_Enabled"
 	1    3700 7300
 	1    0    0    -1
@@
 F 2 "Diode_SMD:D_SOD-323_HandSoldering" H 3700 5950 50  0001 C CNN
 F 3 "~" H 3700 5950 50  0001 C CNN
+F 4 "X" H 3700 5950 50  0001 C CNN "Spice_Primitive"
+F 5 "DI_1N4733A" H 3700 5950 50  0001 C CNN "Spice_Model"
+F 6 "Y" H 3700 5950 50  0001 C CNN "Spice_Netlist_Enabled"
+F 7 "/Users/ihartwig/repos/KiCad-Spice-Library/Models/Diode/zener.lib" H 3700 5950 50  0001 C CNN "Spice_Lib_File"
+F 8 "Nexperia" V 3700 5950 50  0001 C CNN "Mfg"
+F 9 "BZX384-C5V1,115" V 3700 5950 50  0001 C CNN "Mfg PN"
 	1    3700 5950
 	0    1    1    0
@@
 F 6 "Diodes Incorporated" H 3600 4650 50  0001 C CNN "Mfg 2"
 F 7 "DMN5L06DMK-7" H 3600 4650 50  0001 C CNN "Mfg PN 2"
+F 8 "M" H 3600 4650 50  0001 C CNN "Spice_Primitive"
+F 9 "cmosn" H 3600 4650 50  0001 C CNN "Spice_Model"
+F 10 "Y" H 3600 4650 50  0001 C CNN "Spice_Netlist_Enabled"
+F 11 "/Users/ihartwig/repos/KiCad-Spice-Library/Models/Transistor/FET/cmos.lib" H 3600 4650 50  0001 C CNN "Spice_Lib_File"
 	1    3600 4650
 	1    0    0    -1
@@
 F 6 "Diodes Incorporated" H 3600 7000 50  0001 C CNN "Mfg 2"
 F 7 "DMN5L06DMK-7" H 3600 7000 50  0001 C CNN "Mfg PN 2"
+F 8 "M" H 3600 7000 50  0001 C CNN "Spice_Primitive"
+F 9 "cmosn" H 3600 7000 50  0001 C CNN "Spice_Model"
+F 10 "Y" H 3600 7000 50  0001 C CNN "Spice_Netlist_Enabled"
+F 11 "/Users/ihartwig/repos/KiCad-Spice-Library/Models/Transistor/FET/cmos.lib" H 3600 7000 50  0001 C CNN "Spice_Lib_File"
 	2    3600 7000
 	1    0    0    -1
@@
 	2700 6600 2700 7300
 Wire Wire Line
-	2000 5700 2700 5700
-Wire Wire Line
 	3200 6200 3200 7000
 Wire Wire Line
@@
 	3200 3850 3200 4650
 Wire Wire Line
-	2000 3350 2700 3350
+	2000 3350 2100 3350
 Wire Wire Line
 	3700 4350 4150 4350
@@
 Wire Wire Line
 	4150 3350 3700 3350
+$Comp
+L Simulation_SPICE:VDC V_CONN1
+U 1 1 62A3EAB9
+P 1850 4650
+F 0 "V_CONN1" H 1980 4741 50  0000 L CNN
+F 1 "VDC" H 1980 4650 50  0000 L CNN
+F 2 "" H 1850 4650 50  0001 C CNN
+F 3 "~" H 1850 4650 50  0001 C CNN
+F 4 "Y" H 1850 4650 50  0001 L CNN "Spice_Netlist_Enabled"
+F 5 "V" H 1850 4650 50  0001 L CNN "Spice_Primitive"
+F 6 "dc(1)" H 1980 4559 50  0000 L CNN "Spice_Model"
+	1    1850 4650
+	1    0    0    -1
+$EndComp
+Wire Wire Line
+	2300 4950 1850 4950
+Wire Wire Line
+	1850 4950 1850 4850
+Connection ~ 2300 4950
+Wire Wire Line
+	1850 4450 1850 3650
+Wire Wire Line
+	1850 3650 2100 3650
+Wire Wire Line
+	2100 3650 2100 3350
+Connection ~ 2100 3350
+Wire Wire Line
+	2100 3350 2700 3350
+$Comp
+L Simulation_SPICE:VDC V_TR2
+U 1 1 62A55193
+P 1850 7000
+F 0 "V_TR2" H 1980 7091 50  0000 L CNN
+F 1 "VDC" H 1980 7000 50  0000 L CNN
+F 2 "" H 1850 7000 50  0001 C CNN
+F 3 "~" H 1850 7000 50  0001 C CNN
+F 4 "Y" H 1850 7000 50  0001 L CNN "Spice_Netlist_Enabled"
+F 5 "V" H 1850 7000 50  0001 L CNN "Spice_Primitive"
+F 6 "dc(1)" H 1980 6909 50  0000 L CNN "Spice_Model"
+	1    1850 7000
+	1    0    0    -1
+$EndComp
+Wire Wire Line
+	2700 7300 1850 7300
+Wire Wire Line
+	1850 7300 1850 7200
+Connection ~ 2700 7300
+Wire Wire Line
+	2000 5700 2100 5700
+Wire Wire Line
+	1850 6800 1850 6100
+Wire Wire Line
+	1850 6100 2100 6100
+Wire Wire Line
+	2100 6100 2100 5700
+Connection ~ 2100 5700
+Wire Wire Line
+	2100 5700 2700 5700
+$Comp
+L frc-on-ftc-hw-special:R_Pack04_SMD_Split RN1
+U 1 1 626CC9C4
+P 2700 3600
+F 0 "RN1" H 2788 3646 50  0000 L CNN
+F 1 "10k" H 2788 3555 50  0000 L CNN
+F 2 "Resistor_SMD:R_Array_Convex_4x1206" V 2620 3600 50  0001 C CNN
+F 3 "http://www.vishay.com/docs/31509/csc.pdf" H 2700 3600 50  0001 C CNN
+F 4 "Yaego" H 2700 3600 50  0001 C CNN "Mfg"
+F 5 "YC164-JR-0710KL" H 2700 3600 50  0001 C CNN "Mfg PN"
+	1    2700 3600
+	1    0    0    1
+$EndComp
 $EndSCHEMATC

Commit message: add roborio proto r1
Changed lines of the file:
@@
 	1    0    0    1
 $EndComp
+Text Notes 3400 6950 0    50   ~ 0
+Vgs\nMax\n-8V
 $EndSCHEMATC
