File: rio-proto/rio-proto.kicad_pcb (KiCad board)
At the start: 2 copper layers, 25.4 x 31.8 mm, 46 parts, among them J1 Conn_01x02

Commit message: roborio-proto and talonsrx-enc-limit-ftc gerbers again
Other:
- rule pad_to_mask_clearance: 0.05 -> 0.051
