File: talonsrx-enc-limit-ftc/talonsrx-enc-limit-ftc.kicad_pcb (KiCad board)
At the start: 2 copper layers, 43.8 x 27.9 mm, 17 parts, among them J1 Conn_02x05_Odd_Even, J2 Conn_01x04, J3 Conn_01x04, J4 Conn_01x04

Commit message: jetson-nano-ppoe layout r1
Parts:
- moved G*** 3.72 mm to (113.5, 97.2)
Other:
- board text added: "TalonSRX Enc+Lim R1 2022"
- board text added: "ihartwig @ Iron Panthers"
- board text removed: "R1 2022"
- board text removed: "R1 2022 Iron Panthers - FRC 5026"

Commit message: add roborio proto r1
Parts:
- J1: moved to F.Cu
- moved J1 5.08 mm to (149.2, 94.6)
Routing:
- net /+5V: track 34.9 -> 29.6 mm
- net /ENC_A: track 37.9 -> 40.7 mm
- net /LIM_FWD: track 43.4 -> 45.9 mm
- net /+3.3V: track 73.6 -> 71.3 mm
- net /ENC_B: track 38.1 -> 38.9 mm

Commit message: roborio-proto and talonsrx-enc-limit-ftc gerbers again
Other:
- rule pad_to_mask_clearance: 0.05 -> 0.051

Commit message: talonsrx-enc-limit-ftc for jlcpcb asm and fix pinouts
Parts:
- added REF**: MountingHole_1.152mm_JLCPCB_Tooling, frc-on-ftc-hw-special:MountingHole_1.152mm_JLCPCB_Tooling, F.Cu at (145.5, 84.6)
- added REF**: MountingHole_1.152mm_JLCPCB_Tooling, frc-on-ftc-hw-special:MountingHole_1.152mm_JLCPCB_Tooling, F.Cu at (145.5, 109.7)
- added REF**: MountingHole_1.152mm_JLCPCB_Tooling, frc-on-ftc-hw-special:MountingHole_1.152mm_JLCPCB_Tooling, F.Cu at (112.0, 93.0)
- J1: value Conn_02x05_Odd_Even -> DNP
- J2, J3, J4: footprint Connector_JST:JST_PH_B4B-PH-SM4-TB_1x04-1MP_P2.00mm_Vertical -> Connector_JST:JST_PH_S4B-PH-SM4-TB_1x04-1MP_P2.00mm_Horizontal
- REF** (x2): value Zip Tie -> ZT
- moved G*** 32.1 mm to (145.5, 97.9)
- moved REF** 2.69 mm to (113.0, 89.5)
- moved REF** 2.69 mm to (113.0, 104.8)
- moved J2 0.63 mm to (122.6, 90.2), turned to 270 degrees
- moved J3 0.63 mm to (122.6, 104.1), turned to 270 degrees
- moved J4 0.25 mm to (139.3, 101.6), turned to 270 degrees
Connections:
- J2 pad 1: GND -> /ENC_B
- J2 pad 2: /ENC_PWR -> /ENC_A
- J2 pad 3: /ENC_A -> /ENC_PWR
- J2 pad 4: /ENC_B -> GND
- J3 pad 1: GND -> /LIM_REV
- J3 pad 2: /+3.3V -> /LIM_N
- J3 pad 3: /LIM_N -> /+3.3V
- J3 pad 4: Net-(J3-Pad4) -> GND
- J4 pad 1: /LIM_FWD -> /LIM_REV
- J4 pad 4: /LIM_REV -> /LIM_FWD
Routing:
- net (no net): track 0.00 -> 68.7 mm, vias 0 -> 24
- net /LIM_REV: track 36.3 -> 42.9 mm
- net /LIM_FWD: track 45.9 -> 50.3 mm, vias 2 -> 1
- net /ENC_B: track 38.9 -> 34.7 mm
- net /ENC_A: track 40.7 -> 36.5 mm
- net /+3.3V: track 71.3 -> 74.3 mm
- net /LIM_N: track 7.64 -> 6.37 mm
- net /ENC_PWR: track 7.05 -> 6.19 mm
Other:
- outline, holes or cut-outs redrawn
- board text added: "0 1 V G"
- board text added: "B A V G"
- board text added: "R G G F"
