File: talonsrx-enc-limit-ftc/talonsrx-enc-limit-ftc.sch (KiCad schematic (older format))
At the start: 12 parts, among them J1 Conn_02x05_Odd_Even, J2 Conn_01x04, J3 Conn_01x04, J4 Conn_01x04

Commit message: talonsrx-enc-limit-ftc for jlcpcb asm and fix pinouts
Parts:
- D1: JLCPCB PN (none) -> C2293; Mfg (none) -> Hubei Kento Elec; Mfg PN (none) -> C2293
- D2: JLCPCB PN (none) -> C2292; Mfg (none) -> Hubei Kento Elec; Mfg PN (none) -> C2292
- J1: value Conn_02x05_Odd_Even -> DNP; Mfg (none) -> Amphenol CS; Mfg PN (none) -> 20021311-00010T4LF
- J2, J3, J4: footprint Connector_JST:JST_PH_B4B-PH-SM4-TB_1x04-1MP_P2.00mm_Vertical -> Connector_JST:JST_PH_S4B-PH-SM4-TB_1x04-1MP_P2.00mm_Horizontal; JLCPCB PN (none) -> C265332; Mfg (none) -> JST Sales America; Mfg PN (none) -> S4B-PH-SM4-K-TB(LF)(SN)
- R1, R2: JLCPCB PN (none) -> C17520; Mfg (none) -> UNI-ROYAL; Mfg PN (none) -> 0805W8F2201T5E
Connections:
- wire segments 49 -> 50
- no-connect marks 2 -> 1
Changed lines of the file:
@@
 P 4100 2700
 F 0 "J1" H 4150 3117 50  0000 C CNN
-F 1 "Conn_02x05_Odd_Even" H 4150 3026 50  0000 C CNN
+F 1 "DNP" H 4150 3026 50  0000 C CNN
 F 2 "Connector_PinHeader_1.27mm:PinHeader_2x05_P1.27mm_Vertical" H 4100 2700 50  0001 C CNN
 F 3 "~" H 4100 2700 50  0001 C CNN
+F 4 "Amphenol CS" H 4100 2700 50  0001 C CNN "Mfg"
+F 5 "20021311-00010T4LF" H 4100 2700 50  0001 C CNN "Mfg PN"
 	1    4100 2700
 	1    0    0    -1
@@
 L Connector_Generic:Conn_01x04 J2
 U 1 1 625E8CFF
-P 8150 2500
-F 0 "J2" H 8230 2492 50  0000 L CNN
-F 1 "Conn_01x04" H 8230 2401 50  0000 L CNN
-F 2 "Connector_JST:JST_PH_B4B-PH-SM4-TB_1x04-1MP_P2.00mm_Vertical" H 8150 2500 50  0001 C CNN
-F 3 "~" H 8150 2500 50  0001 C CNN
-	1    8150 2500
-	1    0    0    -1
+P 8150 2600
+F 0 "J2" H 8230 2592 50  0000 L CNN
+F 1 "Conn_01x04" H 8230 2501 50  0000 L CNN
+F 2 "Connector_JST:JST_PH_S4B-PH-SM4-TB_1x04-1MP_P2.00mm_Horizontal" H 8150 2600 50  0001 C CNN
+F 3 "~" H 8150 2600 50  0001 C CNN
+F 4 "JST Sales America" H 8150 2600 50  0001 C CNN "Mfg"
+F 5 "S4B-PH-SM4-K-TB(LF)(SN)" H 8150 2600 50  0001 C CNN "Mfg PN"
+F 6 "C265332" H 8150 2600 50  0001 C CNN "JLCPCB PN"
+	1    8150 2600
+	1    0    0    1
 $EndComp
 $Comp
 L Connector_Generic:Conn_01x04 J3
 U 1 1 625E9E4B
-P 8150 3500
-F 0 "J3" H 8230 3492 50  0000 L CNN
-F 1 "Conn_01x04" H 8230 3401 50  0000 L CNN
-F 2 "Connector_JST:JST_PH_B4B-PH-SM4-TB_1x04-1MP_P2.00mm_Vertical" H 8150 3500 50  0001 C CNN
-F 3 "~" H 8150 3500 50  0001 C CNN
-	1    8150 3500
-	1    0    0    -1
+P 8150 3600
+F 0 "J3" H 8230 3592 50  0000 L CNN
+F 1 "Conn_01x04" H 8230 3501 50  0000 L CNN
+F 2 "Connector_JST:JST_PH_S4B-PH-SM4-TB_1x04-1MP_P2.00mm_Horizontal" H 8150 3600 50  0001 C CNN
+F 3 "~" H 8150 3600 50  0001 C CNN
+F 4 "JST Sales America" H 8150 3600 50  0001 C CNN "Mfg"
+F 5 "S4B-PH-SM4-K-TB(LF)(SN)" H 8150 3600 50  0001 C CNN "Mfg PN"
+F 6 "C265332" H 8150 3600 50  0001 C CNN "JLCPCB PN"
+	1    8150 3600
+	1    0    0    1
 $EndComp
 Wire Wire Line
@@
 Text Label 7700 3850 0    50   ~ 0
 LIM_REV
-NoConn ~ 7950 3700
 $Comp
 L Connector_Generic:Conn_01x04 J4
 U 1 1 6260C303
-P 8150 4900
-F 0 "J4" H 8230 4892 50  0000 L CNN
-F 1 "Conn_01x04" H 8230 4801 50  0000 L CNN
-F 2 "Connector_JST:JST_PH_B4B-PH-SM4-TB_1x04-1MP_P2.00mm_Vertical" H 8150 4900 50  0001 C CNN
-F 3 "~" H 8150 4900 50  0001 C CNN
-	1    8150 4900
-	1    0    0    -1
+P 8150 5000
+F 0 "J4" H 8230 4992 50  0000 L CNN
+F 1 "Conn_01x04" H 8230 4901 50  0000 L CNN
+F 2 "Connector_JST:JST_PH_S4B-PH-SM4-TB_1x04-1MP_P2.00mm_Horizontal" H 8150 5000 50  0001 C CNN
+F 3 "~" H 8150 5000 50  0001 C CNN
+F 4 "JST Sales America" H 8150 5000 50  0001 C CNN "Mfg"
+F 5 "S4B-PH-SM4-K-TB(LF)(SN)" H 8150 5000 50  0001 C CNN "Mfg PN"
+F 6 "C265332" H 8150 5000 50  0001 C CNN "JLCPCB PN"
+	1    8150 5000
+	1    0    0    1
 $EndComp
 Text Notes 7000 4550 0    50   ~ 0
@@
 F 2 "LED_SMD:LED_0805_2012Metric" V 4800 4250 50  0001 C CNN
 F 3 "~" V 4800 4250 50  0001 C CNN
+F 4 "Hubei Kento Elec" V 4800 4250 50  0001 C CNN "Mfg"
+F 5 "C2292" V 4800 4250 50  0001 C CNN "Mfg PN"
+F 6 "C2292" V 4800 4250 50  0001 C CNN "JLCPCB PN"
 	1    4800 4250
 	0    -1   -1   0
@@
 F 2 "Resistor_SMD:R_0805_2012Metric" H 4800 3850 50  0001 C CNN
 F 3 "~" H 4800 3850 50  0001 C CNN
+F 4 "UNI-ROYAL" H 4800 3850 50  0001 C CNN "Mfg"
+F 5 "0805W8F2201T5E" H 4800 3850 50  0001 C CNN "Mfg PN"
+F 6 "C17520" H 4800 3850 50  0001 C CNN "JLCPCB PN"
 	1    4800 3850
 	1    0    0    -1
@@
 F 2 "LED_SMD:LED_0805_2012Metric" V 4050 4250 50  0001 C CNN
 F 3 "~" V 4050 4250 50  0001 C CNN
+F 4 "Hubei Kento Elec" V 4050 4250 50  0001 C CNN "Mfg"
+F 5 "C2293" V 4050 4250 50  0001 C CNN "Mfg PN"
+F 6 "C2293" V 4050 4250 50  0001 C CNN "JLCPCB PN"
 	1    4050 4250
 	0    -1   -1   0
@@
 F 2 "Resistor_SMD:R_0805_2012Metric" H 4050 3850 50  0001 C CNN
 F 3 "~" H 4050 3850 50  0001 C CNN
+F 4 "UNI-ROYAL" H 4050 3850 50  0001 C CNN "Mfg"
+F 5 "0805W8F2201T5E" H 4050 3850 50  0001 C CNN "Mfg PN"
+F 6 "C17520" H 4050 3850 50  0001 C CNN "JLCPCB PN"
 	1    4050 3850
 	1    0    0    -1
@@
 Text Label 4800 4050 0    50   ~ 0
 LIM_FWD_A
+Wire Wire Line
+	7600 3700 7950 3700
+Text Label 7600 3700 0    50   ~ 0
+LIM_REV
 $EndSCHEMATC
