File: gigablox-nano-rvp/gigablox-nano-rvp.kicad_sch (KiCad schematic)
At the start: 23 parts, among them IC1 MAX6898AAZT+T, J1 Conn_01x02, J2 Conn_01x03, J3 Conn_01x04, J4 Conn_01x02, Q1 Q_PMOS_GSD, U1 LM4040DIM3-3.0

Commit message: gigablox-nano-rvp floorplan
Parts:
- removed V_CONN1: VDC, symbol Simulation_SPICE:VDC
- added H3: MountingHole, MountingHole:MountingHole_2.2mm_M2, symbol Mechanical:MountingHole
- H1, H2: footprint MountingHole:MountingHole_3.2mm_M3_Pad_Via -> MountingHole:MountingHole_2.2mm_M2
Other:
- note added: "M2 (2.2mm) mounting holes 4.6mm dia hardware clearance 5mm between-board standoff height"
Changed lines of the file:
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@@
   (junction (at 134.62 74.93) (diameter 0) (color 0 0 0 0)
   )
-  (junction (at 55.88 115.57) (diameter 0) (color 0 0 0 0)
-  )
   (junction (at 185.42 157.48) (diameter 0) (color 0 0 0 0)
   )
@@
   )
   (junction (at 66.04 173.99) (diameter 0) (color 0 0 0 0)
-  )
-  (junction (at 50.8 74.93) (diameter 0) (color 0 0 0 0)
   )
   (junction (at 66.04 87.63) (diameter 0) (color 0 0 0 0)
@@
     (stroke (width 0) (type default) (color 0 0 0 0))
   )
-  (wire (pts (xy 44.45 115.57) (xy 44.45 113.03))
-    (stroke (width 0) (type default) (color 0 0 0 0))
-  )
   (wire (pts (xy 91.44 171.45) (xy 91.44 173.99))
     (stroke (width 0) (type default) (color 0 0 0 0))
@@
     (stroke (width 0) (type default) (color 0 0 0 0))
   )
-  (wire (pts (xy 48.26 74.93) (xy 50.8 74.93))
+  (wire (pts (xy 48.26 74.93) (xy 66.04 74.93))
     (stroke (width 0) (type default) (color 0 0 0 0))
   )
@@
     (stroke (width 0) (type default) (color 0 0 0 0))
   )
-  (wire (pts (xy 50.8 74.93) (xy 66.04 74.93))
-    (stroke (width 0) (type default) (color 0 0 0 0))
-  )
   (wire (pts (xy 115.57 149.86) (xy 116.84 149.86))
     (stroke (width 0) (type default) (color 0 0 0 0))
@@
     (stroke (width 0) (type default) (color 0 0 0 0))
   )
-  (wire (pts (xy 44.45 102.87) (xy 44.45 82.55))
-    (stroke (width 0) (type default) (color 0 0 0 0))
-  )
   (wire (pts (xy 81.28 88.9) (xy 81.28 90.17))
     (stroke (width 0) (type default) (color 0 0 0 0))
   )
-  (wire (pts (xy 44.45 82.55) (xy 50.8 82.55))
-    (stroke (width 0) (type default) (color 0 0 0 0))
-  )
   (wire (pts (xy 91.44 147.32) (xy 91.44 148.59))
     (stroke (width 0) (type default) (color 0 0 0 0))
   )
-  (wire (pts (xy 50.8 82.55) (xy 50.8 74.93))
-    (stroke (width 0) (type default) (color 0 0 0 0))
-  )
   (wire (pts (xy 66.04 115.57) (xy 66.04 118.11))
     (stroke (width 0) (type default) (color 0 0 0 0))
@@
   )
   (wire (pts (xy 149.86 77.47) (xy 147.32 77.47))
-    (stroke (width 0) (type default) (color 0 0 0 0))
-  )
-  (wire (pts (xy 55.88 115.57) (xy 44.45 115.57))
     (stroke (width 0) (type default) (color 0 0 0 0))
   )
@@
   (text "IN H & ~{EN} L = ~{OUT} L -> +12V H (On)\n\nIN Rising 0.5V Threshold\n    5.95V nom (5.85-6.06V) after RVP\nIN Falling 0.495V Threshold\n    5.86V nom (5.79-5.99V) after RVP\n\nTdelay = Cdelay * 4e6 + 40usec (in uF)\n    for 0.880 (0.880e6-40us)\n    Cdelay = 0.22uF"
     (at 121.92 185.42 0)
+    (effects (font (size 1.27 1.27)) (justify left bottom))
+  )
+  (text "M2 (2.2mm) mounting holes\n4.6mm dia hardware clearance\n5mm between-board standoff height"
+    (at 231.14 149.86 0)
     (effects (font (size 1.27 1.27)) (justify left bottom))
   )
@@
       (effects (font (size 1.27 1.27)) (justify left))
     )
-    (property "Footprint" "MountingHole:MountingHole_3.2mm_M3_Pad_Via" (id 2) (at 238.76 133.35 0)
+    (property "Footprint" "MountingHole:MountingHole_2.2mm_M2" (id 2) (at 238.76 133.35 0)
       (effects (font (size 1.27 1.27)) hide)
     )
@@
       (effects (font (size 1.27 1.27)) (justify left))
     )
-    (property "Footprint" "MountingHole:MountingHole_3.2mm_M3_Pad_Via" (id 2) (at 238.76 127 0)
+    (property "Footprint" "MountingHole:MountingHole_2.2mm_M2" (id 2) (at 238.76 127 0)
       (effects (font (size 1.27 1.27)) hide)
     )
@@
     (pin "5")
   )
-  (symbol (lib_id "Simulation_SPICE:VDC") (at 44.45 107.95 0) (unit 1)
-    (in_bom yes) (on_board yes)
-    (property "Reference" "V_CONN1" (id 0) (at 47.752 105.6386 0)
-      (effects (font (size 1.27 1.27)) (justify left))
-    )
-    (property "Value" "VDC" (id 1) (at 47.752 107.95 0)
-      (effects (font (size 1.27 1.27)) (justify left))
-    )
-    (property "Footprint" "" (id 2) (at 44.45 107.95 0)
-      (effects (font (size 1.27 1.27)) hide)
-    )
-    (property "Datasheet" "~" (id 3) (at 44.45 107.95 0)
-      (effects (font (size 1.27 1.27)) hide)
-    )
-    (property "Spice_Netlist_Enabled" "Y" (id 4) (at 44.45 107.95 0)
-      (effects (font (size 1.27 1.27)) (justify left) hide)
-    )
-    (property "Spice_Primitive" "V" (id 5) (at 44.45 107.95 0)
-      (effects (font (size 1.27 1.27)) (justify left) hide)
-    )
-    (property "Spice_Model" "dc(1)" (id 6) (at 47.752 110.2614 0)
-      (effects (font (size 1.27 1.27)) (justify left))
-    )
-    (pin "1")
-    (pin "2")
-  )
   (symbol (lib_id "power:GND") (at 242.57 80.01 0) (unit 1)
     (in_bom yes) (on_board yes)
@@
     (pin "1")
     (pin "2")
+  )
+  (symbol (lib_id "Mechanical:MountingHole") (at 238.76 139.7 0) (unit 1)
+    (in_bom yes) (on_board yes)
+    (property "Reference" "H3" (id 0) (at 241.3 138.5316 0)
+      (effects (font (size 1.27 1.27)) (justify left))
+    )
+    (property "Value" "MountingHole" (id 1) (at 241.3 140.843 0)
+      (effects (font (size 1.27 1.27)) (justify left))
+    )
+    (property "Footprint" "MountingHole:MountingHole_2.2mm_M2" (id 2) (at 238.76 139.7 0)
+      (effects (font (size 1.27 1.27)) hide)
+    )
+    (property "Datasheet" "~" (id 3) (at 238.76 139.7 0)
+      (effects (font (size 1.27 1.27)) hide)
+    )
   )
   (symbol (lib_id "power:+3V0") (at 171.45 144.78 0) (unit 1)
@@
     )
     (path "/00000000-0000-0000-0000-00006276e5ce"
-      (reference "H1") (unit 1) (value "MountingHole") (footprint "MountingHole:MountingHole_3.2mm_M3_Pad_Via")
+      (reference "H1") (unit 1) (value "MountingHole") (footprint "MountingHole:MountingHole_2.2mm_M2")
     )
     (path "/00000000-0000-0000-0000-0000626a4a84"
-      (reference "H2") (unit 1) (value "MountingHole") (footprint "MountingHole:MountingHole_3.2mm_M3_Pad_Via")
+      (reference "H2") (unit 1) (value "MountingHole") (footprint "MountingHole:MountingHole_2.2mm_M2")
+    )
+    (path "/210e904d-8097-4da3-900c-7bc86b2bd2a7"
+      (reference "H3") (unit 1) (value "MountingHole") (footprint "MountingHole:MountingHole_2.2mm_M2")
     )
     (path "/9a815496-f5ef-408e-a863-73ffe6d9b091"
@@
       (reference "U1") (unit 1) (value "LM4040DIM3-3.0") (footprint "Package_TO_SOT_SMD:SOT-23")
     )
-    (path "/00000000-0000-0000-0000-000062a3eab9"
-      (reference "V_CONN1") (unit 1) (value "VDC") (footprint "")
-    )
-  )
+  )

Commit message: gigablox-nano-rvp and jetson-nano-ppoe gerbers
Parts:
- added C7: DNP, Capacitor_THT:CP_Radial_D6.3mm_P2.50mm, symbol Device:C_Polarized
Connections:
- net +12V: now also C7.1
- net GND: now also C7.2
Other:
- note added: "Extra holdup caps can work with RVP FET + RST monitor to keep switch operational for short transients under IC1 threshold. Useful range 5.1-5.79V."
- note removed: "Extra holdup caps can work with RVP FET + RST monitor to keep switch operational for short transients under 5.79V after RVP"
- moved on the sheet: J3
Changed lines of the file:
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@@
   (junction (at 185.42 157.48) (diameter 0) (color 0 0 0 0)
   )
-  (junction (at 147.32 82.55) (diameter 0) (color 0 0 0 0)
+  (junction (at 166.37 82.55) (diameter 0) (color 0 0 0 0)
   )
   (junction (at 91.44 185.42) (diameter 0) (color 0 0 0 0)
@@
   (junction (at 80.01 154.94) (diameter 0) (color 0 0 0 0)
   )
+  (junction (at 134.62 86.36) (diameter 0) (color 0 0 0 0)
+  )
   (junction (at 66.04 74.93) (diameter 0) (color 0 0 0 0)
   )
@@
   (junction (at 105.41 185.42) (diameter 0) (color 0 0 0 0)
   )
-  (junction (at 147.32 74.93) (diameter 0) (color 0 0 0 0)
+  (junction (at 146.05 74.93) (diameter 0) (color 0 0 0 0)
+  )
+  (junction (at 166.37 74.93) (diameter 0) (color 0 0 0 0)
   )
   (junction (at 91.44 147.32) (diameter 0) (color 0 0 0 0)
@@
     (stroke (width 0) (type default) (color 0 0 0 0))
   )
+  (wire (pts (xy 123.19 74.93) (xy 134.62 74.93))
+    (stroke (width 0) (type default) (color 0 0 0 0))
+  )
   (wire (pts (xy 91.44 154.94) (xy 91.44 153.67))
     (stroke (width 0) (type default) (color 0 0 0 0))
   )
-  (wire (pts (xy 147.32 77.47) (xy 147.32 74.93))
+  (wire (pts (xy 166.37 77.47) (xy 166.37 74.93))
     (stroke (width 0) (type default) (color 0 0 0 0))
   )
@@
     (stroke (width 0) (type default) (color 0 0 0 0))
   )
+  (wire (pts (xy 146.05 74.93) (xy 146.05 77.47))
+    (stroke (width 0) (type default) (color 0 0 0 0))
+  )
   (wire (pts (xy 185.42 157.48) (xy 185.42 158.75))
     (stroke (width 0) (type default) (color 0 0 0 0))
@@
     (stroke (width 0) (type default) (color 0 0 0 0))
   )
-  (wire (pts (xy 123.19 74.93) (xy 134.62 74.93))
-    (stroke (width 0) (type default) (color 0 0 0 0))
-  )
   (wire (pts (xy 80.01 147.32) (xy 80.01 148.59))
     (stroke (width 0) (type default) (color 0 0 0 0))
@@
     (stroke (width 0) (type default) (color 0 0 0 0))
   )
-  (wire (pts (xy 147.32 80.01) (xy 149.86 80.01))
+  (wire (pts (xy 166.37 80.01) (xy 168.91 80.01))
     (stroke (width 0) (type default) (color 0 0 0 0))
   )
@@
     (stroke (width 0) (type default) (color 0 0 0 0))
   )
-  (wire (pts (xy 147.32 82.55) (xy 144.78 82.55))
+  (wire (pts (xy 166.37 82.55) (xy 163.83 82.55))
     (stroke (width 0) (type default) (color 0 0 0 0))
   )
@@
     (stroke (width 0) (type default) (color 0 0 0 0))
   )
-  (wire (pts (xy 149.86 82.55) (xy 147.32 82.55))
+  (wire (pts (xy 168.91 82.55) (xy 166.37 82.55))
     (stroke (width 0) (type default) (color 0 0 0 0))
   )
@@
     (stroke (width 0) (type default) (color 0 0 0 0))
   )
+  (wire (pts (xy 146.05 86.36) (xy 134.62 86.36))
+    (stroke (width 0) (type default) (color 0 0 0 0))
+  )
   (wire (pts (xy 134.62 74.93) (xy 134.62 78.74))
     (stroke (width 0) (type default) (color 0 0 0 0))
@@
     (stroke (width 0) (type default) (color 0 0 0 0))
   )
+  (wire (pts (xy 146.05 74.93) (xy 166.37 74.93))
+    (stroke (width 0) (type default) (color 0 0 0 0))
+  )
   (wire (pts (xy 66.04 163.83) (xy 66.04 166.37))
     (stroke (width 0) (type default) (color 0 0 0 0))
@@
     (stroke (width 0) (type default) (color 0 0 0 0))
   )
-  (wire (pts (xy 144.78 82.55) (xy 144.78 85.09))
-    (stroke (width 0) (type default) (color 0 0 0 0))
-  )
-  (wire (pts (xy 147.32 74.93) (xy 149.86 74.93))
-    (stroke (width 0) (type default) (color 0 0 0 0))
-  )
-  (wire (pts (xy 134.62 74.93) (xy 147.32 74.93))
+  (wire (pts (xy 134.62 74.93) (xy 146.05 74.93))
+    (stroke (width 0) (type default) (color 0 0 0 0))
+  )
+  (wire (pts (xy 163.83 82.55) (xy 163.83 85.09))
+    (stroke (width 0) (type default) (color 0 0 0 0))
+  )
+  (wire (pts (xy 166.37 74.93) (xy 168.91 74.93))
     (stroke (width 0) (type default) (color 0 0 0 0))
   )
@@
     (stroke (width 0) (type default) (color 0 0 0 0))
   )
-  (wire (pts (xy 147.32 82.55) (xy 147.32 80.01))
+  (wire (pts (xy 166.37 82.55) (xy 166.37 80.01))
     (stroke (width 0) (type default) (color 0 0 0 0))
   )
@@
     (stroke (width 0) (type default) (color 0 0 0 0))
   )
-  (wire (pts (xy 149.86 77.47) (xy 147.32 77.47))
+  (wire (pts (xy 168.91 77.47) (xy 166.37 77.47))
     (stroke (width 0) (type default) (color 0 0 0 0))
   )
@@
   )
   (wire (pts (xy 80.01 154.94) (xy 91.44 154.94))
+    (stroke (width 0) (type default) (color 0 0 0 0))
+  )
+  (wire (pts (xy 146.05 85.09) (xy 146.05 86.36))
     (stroke (width 0) (type default) (color 0 0 0 0))
   )
@@
     (effects (font (size 1.27 1.27)) (justify left bottom))
   )
-  (text "Extra holdup caps can work with\nRVP FET + RST monitor to keep\nswitch operational for short\ntransients under 5.79V after RVP"
+  (text "Extra holdup caps can work with\nRVP FET + RST monitor to keep\nswitch operational for short\ntransients under IC1 threshold.\nUseful range 5.1-5.79V."
     (at 121.92 106.68 0)
     (effects (font (size 1.27 1.27)) (justify left bottom))
@@
   )
   (text "Gigablox Power\nvia 4-pin PicoBlade Cable\n    Molex 0151340400\n5.1 to 60V On"
-    (at 149.86 71.12 0)
+    (at 168.91 71.12 0)
     (effects (font (size 1.27 1.27)) (justify left bottom))
   )
@@
     (effects (font (size 1.27 1.27)) (justify left bottom))
   )
-  (text "Conn Molex 0530470410" (at 149.86 88.9 0)
+  (text "Conn Molex 0530470410" (at 168.91 88.9 0)
     (effects (font (size 1.27 1.27)) (justify left bottom))
   )
@@
     (pin "1")
   )
-  (symbol (lib_id "power:GND") (at 144.78 85.09 0) (unit 1)
-    (in_bom yes) (on_board yes)
-    (property "Reference" "#PWR0109" (id 0) (at 144.78 91.44 0)
-      (effects (font (size 1.27 1.27)) hide)
-    )
-    (property "Value" "GND" (id 1) (at 144.907 89.4842 0))
-    (property "Footprint" "" (id 2) (at 144.78 85.09 0)
-      (effects (font (size 1.27 1.27)) hide)
-    )
-    (property "Datasheet" "" (id 3) (at 144.78 85.09 0)
-      (effects (font (size 1.27 1.27)) hide)
-    )
-    (property "Spice_Primitive" "I" (id 4) (at 144.78 85.09 0)
-      (effects (font (size 1.27 1.27)) hide)
-    )
-    (property "Spice_Netlist_Enabled" "N" (id 5) (at 144.78 85.09 0)
+  (symbol (lib_id "power:GND") (at 163.83 85.09 0) (unit 1)
+    (in_bom yes) (on_board yes)
+    (property "Reference" "#PWR0109" (id 0) (at 163.83 91.44 0)
+      (effects (font (size 1.27 1.27)) hide)
+    )
+    (property "Value" "GND" (id 1) (at 163.957 89.4842 0))
+    (property "Footprint" "" (id 2) (at 163.83 85.09 0)
+      (effects (font (size 1.27 1.27)) hide)
+    )
+    (property "Datasheet" "" (id 3) (at 163.83 85.09 0)
+      (effects (font (size 1.27 1.27)) hide)
+    )
+    (property "Spice_Primitive" "I" (id 4) (at 163.83 85.09 0)
+      (effects (font (size 1.27 1.27)) hide)
+    )
+    (property "Spice_Netlist_Enabled" "N" (id 5) (at 163.83 85.09 0)
       (effects (font (size 1.27 1.27)) hide)
     )
@@
     (pin "5")
   )
+  (symbol (lib_id "Device:C_Polarized") (at 146.05 81.28 0) (unit 1)
+    (in_bom yes) (on_board yes) (fields_autoplaced)
+    (property "Reference" "C7" (id 0) (at 149.86 79.1209 0)
+      (effects (font (size 1.27 1.27)) (justify left))
+    )
+    (property "Value" "DNP" (id 1) (at 149.86 81.6609 0)
+      (effects (font (size 1.27 1.27)) (justify left))
+    )
+    (property "Footprint" "Capacitor_THT:CP_Radial_D6.3mm_P2.50mm" (id 2) (at 147.0152 85.09 0)
+      (effects (font (size 1.27 1.27)) hide)
+    )
+    (property "Datasheet" "~" (id 3) (at 146.05 81.28 0)
+      (effects (font (size 1.27 1.27)) hide)
+    )
+    (pin "1")
+    (pin "2")
+  )
   (symbol (lib_id "power:GND") (at 66.04 186.69 0) (unit 1)
     (in_bom yes) (on_board yes) (fields_autoplaced)
@@
     (pin "2")
   )
-  (symbol (lib_id "Connector_Generic:Conn_01x04") (at 154.94 77.47 0) (unit 1)
-    (in_bom yes) (on_board yes) (fields_autoplaced)
-    (property "Reference" "J3" (id 0) (at 157.48 77.4699 0)
-      (effects (font (size 1.27 1.27)) (justify left))
-    )
-    (property "Value" "Conn_01x04" (id 1) (at 157.48 80.0099 0)
-      (effects (font (size 1.27 1.27)) (justify left))
-    )
-    (property "Footprint" "frc-on-ftc-hw:0530470410" (id 2) (at 154.94 77.47 0)
-      (effects (font (size 1.27 1.27)) hide)
-    )
-    (property "Datasheet" "~" (id 3) (at 154.94 77.47 0)
-      (effects (font (size 1.27 1.27)) hide)
-    )
-    (property "Mfg" "Molex" (id 4) (at 154.94 77.47 0)
-      (effects (font (size 1.27 1.27)) hide)
-    )
-    (property "Mfg PN" "0530470410" (id 5) (at 154.94 77.47 0)
+  (symbol (lib_id "Connector_Generic:Conn_01x04") (at 173.99 77.47 0) (unit 1)
+    (in_bom yes) (on_board yes) (fields_autoplaced)
+    (property "Reference" "J3" (id 0) (at 176.53 77.4699 0)
+      (effects (font (size 1.27 1.27)) (justify left))
+    )
+    (property "Value" "Conn_01x04" (id 1) (at 176.53 80.0099 0)
+      (effects (font (size 1.27 1.27)) (justify left))
+    )
+    (property "Footprint" "frc-on-ftc-hw:0530470410" (id 2) (at 173.99 77.47 0)
+      (effects (font (size 1.27 1.27)) hide)
+    )
+    (property "Datasheet" "~" (id 3) (at 173.99 77.47 0)
+      (effects (font (size 1.27 1.27)) hide)
+    )
+    (property "Mfg" "Molex" (id 4) (at 173.99 77.47 0)
+      (effects (font (size 1.27 1.27)) hide)
+    )
+    (property "Mfg PN" "0530470410" (id 5) (at 173.99 77.47 0)
       (effects (font (size 1.27 1.27)) hide)
     )
@@
       (reference "C6") (unit 1) (value "0.22uF") (footprint "Capacitor_SMD:C_0805_2012Metric")
     )
+    (path "/3128fdb9-a6cc-4120-b6fc-a9c637810477"
+      (reference "C7") (unit 1) (value "DNP") (footprint "Capacitor_THT:CP_Radial_D6.3mm_P2.50mm")
+    )
     (path "/00000000-0000-0000-0000-0000626ca0cd"

Commit message: gigablox-nano-rvp and jetson-nano-ppoe boms
Parts:
- C6: Mfg (none) -> Samsung; Mfg PN (none) -> CL21B224KBFNNNE
- D1: Mfg (none) -> Lite-On; Mfg PN (none) -> LTST-C190GKT
- R1: Mfg (none) -> Yageo; Mfg PN (none) -> RC0603FR-0727KL
- R2: Mfg (none) -> Panasonic; Mfg PN (none) -> ERJ-6GEYJ472V
- R3: Mfg (none) -> Yageo; Mfg PN (none) -> RC0805FR-0724KL
- R4: Mfg (none) -> Yageo; Mfg PN (none) -> RC0805FR-072K2L
Changed lines of the file:
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@@
+      (effects (font (size 1.27 1.27)) hide)
+    )
+    (property "Mfg" "Lite-On" (id 8) (at 102.87 81.28 90)
+      (effects (font (size 1.27 1.27)) hide)
+    )
+    (property "Mfg PN" "LTST-C190GKT" (id 9) (at 102.87 81.28 90)
       (effects (font (size 1.27 1.27)) hide)
     )
@@
       (effects (font (size 1.27 1.27)) hide)
     )
+    (property "Mfg" "" (id 4) (at 105.41 180.34 0)
+      (effects (font (size 1.27 1.27)) hide)
+    )
     (pin "1")
     (pin "2")
@@
       (effects (font (size 1.27 1.27)) hide)
     )
+    (property "Mfg" "Yageo" (id 4) (at 91.44 168.91 0)
+      (effects (font (size 1.27 1.27)) hide)
+    )
+    (property "Mfg PN" "RC0805FR-0724KL" (id 5) (at 91.44 168.91 0)
+      (effects (font (size 1.27 1.27)) hide)
+    )
     (pin "1")
     (pin "2")
@@
       (effects (font (size 1.27 1.27)) hide)
     )
+    (property "Mfg" "Yageo" (id 4) (at 66.04 168.91 0)
+      (effects (font (size 1.27 1.27)) hide)
+    )
+    (property "Mfg PN" "RC0603FR-0727KL" (id 5) (at 66.04 168.91 0)
+      (effects (font (size 1.27 1.27)) hide)
+    )
     (pin "1")
     (pin "2")
@@
     )
     (property "Datasheet" "~" (id 3) (at 185.42 152.4 0)
+      (effects (font (size 1.27 1.27)) hide)
+    )
+    (property "Mfg" "Samsung" (id 4) (at 185.42 152.4 0)
+      (effects (font (size 1.27 1.27)) hide)
+    )
+    (property "Mfg PN" "CL21B224KBFNNNE" (id 5) (at 185.42 152.4 0)
       (effects (font (size 1.27 1.27)) hide)
     )
@@
       (effects (font (size 1.27 1.27)) hide)
     )
+    (property "Mfg" "Panasonic" (id 4) (at 80.01 151.13 0)
+      (effects (font (size 1.27 1.27)) hide)
+    )
+    (property "Mfg PN" "ERJ-6GEYJ472V" (id 5) (at 80.01 151.13 0)
+      (effects (font (size 1.27 1.27)) hide)
+    )
     (pin "1")
     (pin "2")
@@
       (effects (font (size 1.27 1.27)) hide)
     )
+    (property "Mfg" "Yageo" (id 4) (at 91.44 180.34 0)
+      (effects (font (size 1.27 1.27)) hide)
+    )
+    (property "Mfg PN" "RC0805FR-072K2L" (id 5) (at 91.44 180.34 0)
+      (effects (font (size 1.27 1.27)) hide)
+    )
